File: Arduino_Pro_Mini_Dx.kicad_pcb (KiCad board)
At the start: 2 copper layers, 17.8 x 33 mm, 26 parts, among them M1 Arduino Pro Mini Dx, SW1 Reset, U1 AVR128DB32x-xRXB, Y1 32.768kHz

Commit message: project files updated to Kicad version 9.0.1
Other:
- board text added: "Arduino Pro Mini Dx v${REVISION}"
- board text removed: "Arduino Pro Mini Dx v1.0"
