File: Arduino_Pro_Mini_Dx.kicad_sch (KiCad schematic)
At the start: 26 parts, among them M1 Arduino Pro Mini Dx, SW1 Reset, U1 AVR128DB32x-xRXB, Y1 32.768kHz

Commit message: project files updated to Kicad version 9.0.1
Parts:
- renumbered C1 to C10, C1 to C11, C1 to C12, C1 to C13, C1 to C5, C1 to C6, C1 to C7, C1 to C8, C1 to C9, R8 to R1, R8 to R2, R8 to R3
Changed lines of the file:
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@@
 (kicad_sch
-	(version 20231120)
+	(version 20250114)
 	(generator "eeschema")
-	(generator_version "8.0")
+	(generator_version "9.0")
 	(paper "A4")
 	(title_block
@@
 	(label "PA2"
 		(at 234.95 81.28 0)
-		(fields_autoplaced yes)
 		(effects
 			(font
@@
 	(label "PC3"
 		(at 191.77 99.06 180)
-		(fields_autoplaced yes)
 		(effects
 			(font
@@
 	(label "PA7"
 		(at 87.63 133.35 180)
-		(fields_autoplaced yes)
 		(effects
 			(font
@@
 	(label "PC0"
 		(at 142.24 100.33 0)
-		(fields_autoplaced yes)
 		(effects
 			(font
@@
 	(label "PF2"
 		(at 191.77 88.9 180)
-		(fields_autoplaced yes)
 		(effects
 			(font
@@
 	(label "PA6"
 		(at 142.24 92.71 0)
-		(fields_autoplaced yes)
 		(effects
 			(font
@@
 	(label "PD4"
 		(at 234.95 96.52 0)
-		(fields_autoplaced yes)
 		(effects
 			(font
@@
 	(label "PF3"
 		(at 191.77 91.44 180)
-		(fields_autoplaced yes)
 		(effects
 			(font
@@
 	(label "PD3"
 		(at 101.6 107.95 180)
-		(fields_autoplaced yes)
 		(effects
 			(font
@@
 	(label "PA1"
 		(at 191.77 81.28 180)
-		(fields_autoplaced yes)
 		(effects
 			(font
@@
 	(label "PC1"
 		(at 142.24 102.87 0)
-		(fields_autoplaced yes)
 		(effects
 			(font
@@
 	(label "PA5"
 		(at 234.95 109.22 0)
-		(fields_autoplaced yes)
 		(effects
 			(font
@@
 	(label "PA0"
 		(at 142.24 77.47 0)
-		(fields_autoplaced yes)
 		(effects
 			(font
@@
 	(label "PC1"
 		(at 191.77 104.14 180)
-		(fields_autoplaced yes)
 		(effects
 			(font
@@
 	(label "PD1"
 		(at 101.6 102.87 180)
-		(fields_autoplaced yes)
 		(effects
 			(font
@@
 	(label "PC2"
 		(at 191.77 101.6 180)
-		(fields_autoplaced yes)
 		(effects
 			(font
@@
 	(label "PC0"
 		(at 191.77 106.68 180)
-		(fields_autoplaced yes)
 		(effects
 			(font
@@
 	(label "PD1"
 		(at 234.95 104.14 0)
-		(fields_autoplaced yes)
 		(effects
 			(font
@@
 	(label "PD7"
 		(at 101.6 118.11 180)
-		(fields_autoplaced yes)
 		(effects
 			(font
@@
 	(label "PA2"
 		(at 142.24 82.55 0)
-		(fields_autoplaced yes)
 		(effects
 			(font
@@
 	(label "PA3"
 		(at 142.24 85.09 0)
-		(fields_autoplaced yes)
 		(effects
 			(font
@@
 	(label "PA7"
 		(at 142.24 95.25 0)
-		(fields_autoplaced yes)
 		(effects
 			(font
@@
 	(label "PD4"
 		(at 101.6 110.49 180)
-		(fields_autoplaced yes)
 		(effects
 			(font
@@
 	(label "PD7"
 		(at 191.77 116.84 180)
-		(fields_autoplaced yes)
 		(effects
 			(font
@@
 	(label "PD6"
 		(at 191.77 114.3 180)
-		(fields_autoplaced yes)
 		(effects
 			(font
@@
 	(label "PF3"
 		(at 101.6 90.17 180)
-		(fields_autoplaced yes)
 		(effects
 			(font
@@
 	(label "PA3"
 		(at 234.95 78.74 0)
-		(fields_autoplaced yes)
 		(effects
 			(font
@@
 	(label "PA1"
 		(at 142.24 80.01 0)
-		(fields_autoplaced yes)
 		(effects
 			(font
@@
 	(label "PA7"
 		(at 234.95 114.3 0)
-		(fields_autoplaced yes)
 		(effects
 			(font
@@
 	(label "PA4"
 		(at 234.95 111.76 0)
-		(fields_autoplaced yes)
 		(effects
 			(font
@@
 	(label "PA4"
 		(at 142.24 87.63 0)
-		(fields_autoplaced yes)
 		(effects
 			(font
@@
 	(label "PD3"
 		(at 234.95 99.06 0)
-		(fields_autoplaced yes)
 		(effects
 			(font
@@
 	(label "PF2"
 		(at 101.6 87.63 180)
-		(fields_autoplaced yes)
 		(effects
 			(font
@@
 	(label "PA0"
 		(at 191.77 78.74 180)
-		(fields_autoplaced yes)
 		(effects
 			(font
@@
 	(label "PC3"
 		(at 142.24 107.95 0)
-		(fields_autoplaced yes)
 		(effects
 			(font
@@
 	(label "PF4"
 		(at 191.77 93.98 180)
-		(fields_autoplaced yes)
 		(effects
 			(font
@@
 	(label "PD5"
 		(at 191.77 111.76 180)
-		(fields_autoplaced yes)
 		(effects
 			(font
@@
 	(label "PD2"
 		(at 101.6 105.41 180)
-		(fields_autoplaced yes)
 		(effects
 			(font
@@
 	(label "PF5"
 		(at 101.6 95.25 180)
-		(fields_autoplaced yes)
 		(effects
 			(font
@@
 	(label "PD2"
 		(at 234.95 101.6 0)
-		(fields_autoplaced yes)
 		(effects
 			(font
@@
 	(label "PF4"
 		(at 101.6 92.71 180)
-		(fields_autoplaced yes)
 		(effects
 			(font
@@
 	(label "PA6"
 		(at 234.95 106.68 0)
-		(fields_autoplaced yes)
 		(effects
 			(font
@@
 	(label "PD6"
 		(at 101.6 115.57 180)
-		(fields_autoplaced yes)
 		(effects
 			(font
@@
 	(label "PF5"
 		(at 191.77 96.52 180)
-		(fields_autoplaced yes)
 		(effects
 			(font
@@
 	(label "PA5"
 		(at 142.24 90.17 0)
-		(fields_autoplaced yes)
 		(effects
 			(font
@@
 	(label "PD5"
 		(at 101.6 113.03 180)
-		(fields_autoplaced yes)
 		(effects
 			(font
@@
 	(label "PC2"
 		(at 142.24 105.41 0)
-		(fields_autoplaced yes)
 		(effects
 			(font
@@
 		(on_board yes)
 		(dnp no)
-		(property "Reference" "C1"
+		(property "Reference" "C11"
 			(at 130.81 59.69 0)
 			(effects
@@
 		(on_board yes)
 		(dnp no)
-		(property "Reference" "#PWR0103"
+		(property "Reference" "#PWR02"
 			(at 121.92 166.37 0)
 			(effects
@@
 		(on_board yes)
 		(dnp no)
-		(property "Reference" "C1"
+		(property "Reference" "C13"
 			(at 146.05 59.69 0)
 			(effects
@@
 		(on_board yes)
 		(dnp no)
-		(property "Reference" "C1"
+		(property "Reference" "C5"
 			(at 50.8 152.4 0)
 			(effects
@@
 		(on_board yes)
 		(dnp no)
-		(property "Reference" "C1"
+		(property "Reference" "C8"
 			(at 123.19 153.67 0)
 			(effects
@@
 		(on_board yes)
 		(dnp no)
-		(property "Reference" "C1"
+		(property "Reference" "C9"
 			(at 130.81 153.67 0)
 			(effects
@@
 		(on_board yes)
 		(dnp no)
-		(property "Reference" "#PWR0103"
+		(property "Reference" "#PWR04"
 			(at 64.77 102.87 0)
 			(effects
@@
 		(on_board yes)
 		(dnp no)
-		(property "Reference" "R8"
+		(property "Reference" "R1"
 			(at 40.64 146.05 90)
 			(effects
@@
 		(on_board yes)
 		(dnp no)
-		(property "Reference" "R8"
+		(property "Reference" "R3"
 			(at 80.01 76.2 90)
 			(effects
@@
 		(on_board yes)
 		(dnp no)
-		(property "Reference" "C1"
+		(property "Reference" "C10"
 			(at 138.43 153.67 0)
 			(effects
@@
 		(on_board yes)
 		(dnp no)
-		(property "Reference" "R8"
+		(property "Reference" "R2"
 			(at 51.308 139.8016 0)
 			(effects
@@
 		(on_board yes)
 		(dnp no)
-		(property "Reference" "C1"
+		(property "Reference" "C12"
 			(at 138.43 59.69 0)
 			(effects
@@
 		(on_board yes)
 		(dnp no)
-		(property "Reference" "#PWR0103"
+		(property "Reference" "#PWR020"
 			(at 144.78 72.39 0)
 			(effects
@@
 		(on_board yes)
 		(dnp no)
-		(property "Reference" "#PWR0103"
+		(property "Reference" "#PWR06"
 			(at 49.53 166.37 0)
 			(effects
@@
 		(on_board yes)
 		(dnp no)
-		(property "Reference" "#PWR0103"
+		(property "Reference" "#PWR017"
 			(at 121.92 134.62 0)
 			(effects
@@
 		(on_board yes)
 		(dnp no)
-		(property "Reference" "#PWR0103"
+		(property "Reference" "#PWR011"
 			(at 213.36 59.69 0)
 			(effects
@@
 		(on_board yes)
 		(dnp no)
-		(property "Reference" "#PWR0103"
+		(property "Reference" "#PWR012"
 			(at 245.11 88.9 0)
 			(effects
@@
 		(on_board yes)
 		(dnp no)
-		(property "Reference" "C1"
+		(property "Reference" "C6"
 			(at 107.95 153.67 0)
 			(effects
@@
 		(on_board yes)
 		(dnp no)
-		(property "Reference" "#PWR0103"
+		(property "Reference" "#PWR07"
 			(at 38.1 166.37 0)
 			(effects
@@
 		(on_board yes)
 		(dnp no)
-		(property "Reference" "C1"
+		(property "Reference" "C7"
 			(at 115.57 153.67 0)
 			(effects
@@
 		(on_board yes)
 		(dnp no)
-		(property "Reference" "#PWR0103"
+		(property "Reference" "#PWR013"
 			(at 181.61 86.36 0)
 			(effects
@@
 		(on_board yes)
 		(dnp no)
-		(property "Reference" "#PWR0103"
+		(property "Reference" "#PWR018"
 			(at 190.5 127 0)
 			(effects
@@
 		)
 	)
+	(embedded_fonts no)
 )
